File: electronics/cube/cube.kicad_pcb (KiCad board)
At the start: 2 copper layers, 50 x 50 mm, 14 parts, among them J1 Conn_01x02_Male, J2 Conn_01x04_Male, J3 Conn_01x06_Male, J4 Conn_01x02_Male, J5 Conn_01x02_Male, J6 Conn_01x04_Female, J7 Conn_01x02_Male, J8 Conn_01x02_Male, U1 MX1508

Commit message: added holes
Parts:
- added H1: MountingHole, MountingHole:MountingHole_2.2mm_M2_Pad_Via, F.Cu at (193.4, 60.1)
- added H2: MountingHole, MountingHole:MountingHole_2.2mm_M2_Pad_Via, F.Cu at (153.4, 100.1)
- added H3: MountingHole, MountingHole:MountingHole_2.2mm_M2_Pad_Via, F.Cu at (153.4, 60.1)
- added H4: MountingHole, MountingHole:MountingHole_2.2mm_M2_Pad_Via, F.Cu at (193.4, 100.1)
- moved D1 4.19 mm to (161.0, 99.9)
- moved J3 1.90 mm to (194.0, 66.1)
Routing:
- net VCC: track 168.6 -> 165.4 mm
- net /MAIN_UART_TX: track 10.9 -> 8.98 mm
- net /MAIN_UART_RX: track 11.4 -> 9.50 mm
- net /BOOT: track 14.2 -> 12.3 mm
- net +3V3: track 49.3 -> 47.4 mm
- net VDD: track 65.8 -> 66.8 mm

Commit message: Added features + bugfixes
Parts:
- added C3: 4.7uF, Capacitor_SMD:C_0603_1608Metric_Pad1.08x0.95mm_HandSolder, F.Cu at (182.6, 98.0)
- added C4: 4.7uF, Capacitor_SMD:C_0603_1608Metric_Pad1.08x0.95mm_HandSolder, B.Cu at (189.3, 84.4)
- added C5: 0.1uF, Capacitor_SMD:C_0603_1608Metric_Pad1.08x0.95mm_HandSolder, F.Cu at (191.3, 76.6)
- added C6: 10uF, Capacitor_SMD:C_0603_1608Metric_Pad1.08x0.95mm_HandSolder, F.Cu at (161.6, 75.2)
- added C7: 10uF, Capacitor_SMD:C_0603_1608Metric_Pad1.08x0.95mm_HandSolder, F.Cu at (161.7, 69.6)
- added C8: 0.1uF, Capacitor_SMD:C_0603_1608Metric_Pad1.08x0.95mm_HandSolder, F.Cu at (161.6, 72.6)
- added PS1: AP2114HA-3.3TRG1, Package_TO_SOT_SMD:SOT-223-3_TabPin2, F.Cu at (153.8, 76.3)
- added R2: 10k, Resistor_SMD:R_0603_1608Metric_Pad0.98x0.95mm_HandSolder, F.Cu at (191.2, 74.3)
- added R3: 1k, Resistor_SMD:R_0603_1608Metric_Pad0.98x0.95mm_HandSolder, F.Cu at (188.1, 79.3)
- added R4: 2.55k, Resistor_SMD:R_0603_1608Metric_Pad0.98x0.95mm_HandSolder, F.Cu at (158.1, 61.9)
- added R5: 2.55k, Resistor_SMD:R_0603_1608Metric_Pad0.98x0.95mm_HandSolder, F.Cu at (162.6, 62.1)
- moved J1 45.9 mm to (186.4, 97.3), turned to 90 degrees
- moved J2 45.4 mm to (158.3, 58.1), turned to 90 degrees
- moved J4 44.1 mm to (194.4, 66.5), turned to 0 degrees
- moved C1 42.0 mm to (189.8, 90.1)
- moved J6 36.2 mm to (170.5, 58.1), turned to 90 degrees
- moved J5 36.1 mm to (189.9, 66.5), turned to 0 degrees
- moved J8 34.3 mm to (183.8, 102.3), turned to 90 degrees
- moved J7 24.3 mm to (163.4, 101.8), turned to 90 degrees
- moved U1 24.1 mm to (175.0, 100.6), turned to -90 degrees
- moved R1 16.0 mm to (151.3, 87.5), turned to -90 degrees
- moved D1 14.2 mm to (155.2, 87.0), turned to 90 degrees
- moved J3 8.24 mm to (195.6, 74.2)
- moved A1 4.48 mm to (174.2, 77.9)
- moved C2 2.81 mm to (155.9, 93.5)
Connections:
- A1 pad 18: unconnected-(A1-Pad18) -> /Echo
- A1 pad 25: /BOOT -> Net-(A1-Pad25)
- A1 pad 5: unconnected-(A1-Pad5) -> /Trig
- J2 pad 3: VCC -> +3V3
Routing:
- net /SDA: track 5.85 -> 71.0 mm, vias 0 -> 1
- net +3V3: track 47.4 -> 107.5 mm
- net /SCL: track 5.33 -> 64.2 mm, vias 0 -> 1
- net /Echo: track 0.00 -> 45.7 mm, vias 0 -> 1
- net VCC: track 165.4 -> 129.1 mm
- net /Trig: track 0.00 -> 35.5 mm, vias 0 -> 1
- net VDD: track 66.8 -> 41.2 mm, vias 2 -> 0
- net /INB2: track 7.45 -> 30.9 mm
- net /INA2: track 7.45 -> 30.8 mm
- net /INB1: track 10.4 -> 32.5 mm
- net /INA1: track 10.4 -> 30.4 mm
- net /RESET: track 50.0 -> 69.9 mm, vias 0 -> 1
- net Net-(A1-Pad25): track 0.00 -> 9.72 mm
- net /OUTA2: track 4.99 -> 13.9 mm
- net +BATT: track 13.1 -> 4.46 mm
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- removed copper zone on B.Cu, net GND
- removed copper zone on F.Cu, net GND
